File: kicad/Digital Audio Switch.kicad_pcb (KiCad board)
At the start: 2 copper layers, 124.5 x 78.7 mm, 11 parts, among them J1 LINE 1, J2 LINE OUT, J3 LINE 2, J4 PHONO L, J5 PHONO R, J6 OLED I2C, SW1 ROTARY, U1 MCP4231, U2 ESP32, U3 4052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

Commit message: Polish PCB design
Parts:
- added H1: MountingHole_3.2mm_M3, MountingHole:MountingHole_3.2mm_M3, F.Cu at (176.5, 66.0)
- added H2: MountingHole_3.2mm_M3, MountingHole:MountingHole_3.2mm_M3, F.Cu at (86.4, 66.0)
- added H3: MountingHole_3.2mm_M3, MountingHole:MountingHole_3.2mm_M3, F.Cu at (77.5, 120.7)
- added H4: MountingHole_3.2mm_M3, MountingHole:MountingHole_3.2mm_M3, F.Cu at (172.7, 130.8)
- J1, J2, J3: footprint Connector_Audio:Jack_3.5mm_CUI_SJ1-3533NG_Horizontal -> Digital Audio Switch:Jack_3.5mm_CUI_SJ1-3533NG_Horizontal
- J6: footprint Connector_PinHeader_2.54mm:PinHeader_1x04_P2.54mm_Vertical -> Digital Audio Switch:I2C Pin Header
- moved J4 9.56 mm to (100.3, 64.7)
- moved J5 9.56 mm to (115.6, 64.7)
- moved J1 4.04 mm to (76.2, 62.2)
- moved J2 4.04 mm to (189.8, 62.2)
- moved J3 3.59 mm to (190.0, 135.9)
Routing:
- net GND: track 169.0 -> 187.4 mm, vias 0 -> 1
- net GNDA: track 233.8 -> 248.5 mm
- net Net-(U3-Y1): track 83.5 -> 95.5 mm, vias 0 -> 1
- net Net-(J5-In): track 15.2 -> 24.7 mm
- net Net-(U1-PA0): track 86.6 -> 77.2 mm, vias 1 -> 2
- net Net-(U3-Y3): track 34.1 -> 39.3 mm
- net Net-(U2-IO23): track 26.9 -> 21.9 mm
- net Net-(U1-PW0): track 37.7 -> 41.8 mm
- net Net-(U3-X1): track 80.0 -> 84.0 mm
- net Net-(U3-Y0): track 51.1 -> 52.8 mm
- net Net-(J4-In): track 40.1 -> 41.7 mm
- net Net-(U3-X3): track 48.9 -> 47.2 mm
- net Net-(U2-IO25): track 58.4 -> 59.3 mm
- net VCC: track 151.4 -> 150.9 mm
- net Net-(J6-Pin_1): track 47.9 -> 47.6 mm, vias 1 -> 0
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Other:
- board text added: "Digital Audio Switch & Volume Control Hardware Revision v1 by Correl Roush"
- board text added: "JLCJLCJLCJLC"
- board text removed: "LINE 2"
