File: kicad/Digital Audio Switch.kicad_pcb (KiCad board)
At the start: 2 copper layers, 124.5 x 78.7 mm, 15 parts, among them J1 LINE 1, J2 LINE OUT, J3 LINE 2, J4 PHONO L, J5 PHONO R, J6 OLED I2C, SW1 ROTARY, U1 MCP4231, U2 ESP32, U3 4052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

Commit message: Add additional part models
Parts:
- SW1: footprint Rotary_Encoder:RotaryEncoder_Bourns_Horizontal_PEC12R-2xxxF-Sxxxx -> Digital Audio Switch:RotaryEncoder_Bourns_Horizontal_PEC12R-2xxxF-Sxxxx
Changed lines of the file:
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@@
       (rotate (xyz 0 180 0))
     )
-    (model "${VL_PACKAGES3D}/esp32_devkit_v1_doit.3dshapes/esp32_devkit_v1_doit.step"
+    (model "${KIPRJMOD}/esp32_devkit_v1_doit.step"
       (offset (xyz -12.7 0 2.5))
       (scale (xyz 1 1 1))
@@
     (property "ki_keywords" "BNC SMA SMB SMC LEMO coaxial connector CINCH RCA")
     (attr through_hole)
-    (fp_text reference "J4" (at -2.54 -7.62 -90) (layer "F.Fab")
+    (fp_text reference "J4" (at -2.54 -7.62 90) (layer "F.Fab")
         (effects (font (size 1.524 1.524) (thickness 0.3048)))
     )
-    (fp_text value "PHONO L" (at 2.54 7.62 -90) (layer "F.SilkS")
+    (fp_text value "PHONO L" (at 2.54 7.62 90) (layer "F.SilkS")
         (effects (font (size 1.524 1.524) (thickness 0.3048)))
     )
@@
     (pad "2" thru_hole oval (at 0 0 270) (size 4 5.5) (drill 3.3) (layers "*.Cu" "*.Mask")
       (net 2 "GNDA") (pinfunction "Ext") (pintype "passive"))
+    (model "${KIPRJMOD}/KLPX-0848A-2-x.IGS"
+      (offset (xyz -4.5 0 0))
+      (scale (xyz 1 1 1))
+      (rotate (xyz -90 0 90))
+    )
   )
   (footprint "Digital Audio Switch:PCM5102" (layer "F.Cu")
@@
     (pad "" np_thru_hole circle (at 0 0) (size 3.2 3.2) (drill 3.2) (layers "*.Cu" "*.Mask"))
   )
-  (footprint "Rotary_Encoder:RotaryEncoder_Bourns_Horizontal_PEC12R-2xxxF-Sxxxx" (layer "F.Cu")
+  (footprint "Digital Audio Switch:RotaryEncoder_Bourns_Horizontal_PEC12R-2xxxF-Sxxxx" (layer "F.Cu")
     (at 76.28 135.615 -90)
     (descr "Bourns rotary encoder, PEC12R, with switch, horizontal shaft, https://www.bourns.com/docs/product-datasheets/pec12r.pdf")
@@
     (property "ki_keywords" "rotary switch encoder switch push button")
     (attr through_hole)
-    (fp_text reference "SW1" (at -4.7 -2.5 180) (layer "F.SilkS")
+    (fp_text reference "SW1" (at -4.7 -2.5) (layer "F.SilkS")
         (effects (font (size 1 1) (thickness 0.16)))
     )
@@
         (effects (font (size 1 1) (thickness 0.15)))
     )
-    (fp_text user "${REFERENCE}" (at -1.3 -2.5 180) (layer "F.Fab")
+    (fp_text user "${REFERENCE}" (at -1.3 -2.5) (layer "F.Fab")
         (effects (font (size 1 1) (thickness 0.15)))
     )
@@
     (pad "SH" thru_hole roundrect (at -3.5 -7.9) (size 2.9 2.8) (drill oval 2.1 2) (layers "*.Cu" "*.Mask") (roundrect_rratio 0.25))
     (pad "SH" thru_hole roundrect (at -3.5 2.9) (size 2.9 2.8) (drill oval 2.1 2) (layers "*.Cu" "*.Mask") (roundrect_rratio 0.25))
-    (model "${KICAD6_3DMODEL_DIR}/Rotary_Encoder.3dshapes/RotaryEncoder_Bourns_Horizontal_PEC12R-2xxxF-Sxxxx.wrl"
-      (offset (xyz 0 0 0))
-      (scale (xyz 1 1 1))
-      (rotate (xyz 0 0 0))
+    (model "${KIPRJMOD}/PEC12R-2220F-S0024--3DModel-STEP-1.STEP"
+      (offset (xyz -3.5 2.5 0))
+      (scale (xyz 1 1 1))
+      (rotate (xyz -90 0 -90))
     )
   )
@@
     (pad "2" thru_hole oval (at 0 0 270) (size 4 5.5) (drill 3.3) (layers "*.Cu" "*.Mask")
       (net 2 "GNDA") (pinfunction "Ext") (pintype "passive"))
+    (model "${KIPRJMOD}/KLPX-0848A-2-x.IGS"
+      (offset (xyz -4.5 0 0))
+      (scale (xyz 1 1 1))
+      (rotate (xyz -90 0 90))
+    )
   )
   (footprint "Digital Audio Switch:I2C Pin Header" (layer "F.Cu")
