File: kicad/Digital Audio Switch.kicad_sch (KiCad schematic)
At the start: 11 parts, among them J1 LINE 1, J2 LINE OUT, J3 LINE 2, J4 PHONO L, J5 PHONO R, J6 OLED I2C, SW1 ROTARY, U1 MCP4231, U2 ESP32, U3 4052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

Commit message: Polish PCB design
Parts:
- J1, J2, J3: footprint Connector_Audio:Jack_3.5mm_CUI_SJ1-3533NG_Horizontal -> Digital Audio Switch:Jack_3.5mm_CUI_SJ1-3533NG_Horizontal
- J6: footprint Connector_PinHeader_2.54mm:PinHeader_1x04_P2.54mm_Vertical -> Digital Audio Switch:I2C Pin Header
Changed lines of the file:
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@@
       (effects (font (size 1.27 1.27)) (justify left))
     )
-    (property "Footprint" "Connector_PinHeader_2.54mm:PinHeader_1x04_P2.54mm_Vertical" (at 181.61 135.89 0)
+    (property "Footprint" "Digital Audio Switch:I2C Pin Header" (at 181.61 135.89 0)
       (effects (font (size 1.27 1.27)) hide)
     )
@@
       (effects (font (size 1.27 1.27)))
     )
-    (property "Footprint" "Connector_Audio:Jack_3.5mm_CUI_SJ1-3533NG_Horizontal" (at 241.3 60.96 0)
+    (property "Footprint" "Digital Audio Switch:Jack_3.5mm_CUI_SJ1-3533NG_Horizontal" (at 241.3 60.96 0)
       (effects (font (size 1.27 1.27)) hide)
     )
@@
       (effects (font (size 1.27 1.27)))
     )
-    (property "Footprint" "Connector_Audio:Jack_3.5mm_CUI_SJ1-3533NG_Horizontal" (at 43.18 31.75 0)
+    (property "Footprint" "Digital Audio Switch:Jack_3.5mm_CUI_SJ1-3533NG_Horizontal" (at 43.18 31.75 0)
       (effects (font (size 1.27 1.27)) hide)
     )
@@
       (effects (font (size 1.27 1.27)))
     )
-    (property "Footprint" "Connector_Audio:Jack_3.5mm_CUI_SJ1-3533NG_Horizontal" (at 43.18 46.99 0)
-      (effects (font (size 1.27 1.27)) hide)
-    )
+    (property "Footprint" "Digital Audio Switch:Jack_3.5mm_CUI_SJ1-3533NG_Horizontal" (at 43.18 46.99 0)
+      (effects (font (size 1.27 1.27)) hide)
+    )

Commit message: Add additional part models
Parts:
- SW1: footprint Rotary_Encoder:RotaryEncoder_Bourns_Horizontal_PEC12R-2xxxF-Sxxxx -> Digital Audio Switch:RotaryEncoder_Bourns_Horizontal_PEC12R-2xxxF-Sxxxx
Changed lines of the file:
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@@
       (effects (font (size 1.27 1.27)) (justify left))
     )
-    (property "Footprint" "Rotary_Encoder:RotaryEncoder_Bourns_Horizontal_PEC12R-2xxxF-Sxxxx" (at 26.924 182.88 0)
+    (property "Footprint" "Digital Audio Switch:RotaryEncoder_Bourns_Horizontal_PEC12R-2xxxF-Sxxxx" (at 26.924 182.88 0)
       (effects (font (size 1.27 1.27)) hide)
     )
